File: tia-fpga.kicad_sch (KiCad schematic)
At the start: 22 parts, among them J1 Tang Nano 9K row A, J2 TIA pins 1-20, J3 TIA pins 21-40, J4 Tang Nano 9K row B, U1 74AHCT125, U2 74LVC245A, U3 74LVC541A, U4 74LVC541A

Commit message: Use the verified Tang Nano 9K pin map; rework the bus control to fit
The header pinout was read off both revisions of the official Sipeed board
schematic (Tang_Nano_9k_3672 and Tang_nano_9K_3674), which agree exactly.
Two things came out of that, and the second one changed the design.

The headers are 2x24, not 2x20 as previously drawn. J1/J4 are now
Conn_01x24 with every pin accounted for.

Of the 48 header pins only 29 are usable 3.3 V GPIO:

  22  J5/1-22                 banks 1/2 at 3.3 V
   7  J6/1,10,11,19-22        3.3 V
   8  J6/2-9                  BANK3 at 1.8 V - NOT usable at 3.3 V
   8  J5/23-24, J6/12-17      HDMI differential pairs, not GPIO
   3  J6/18,23,24             power

Rev A as drawn needed 30, so it was one pin over. Fixed by taking both
74LVC245 control lines off the FPGA: the A side now faces the FPGA, which
lets DIR be driven straight from the buffered R/W (DIR=1, a read, sends
FPGA -> TIA), and /OE comes from a new 74LVC1G32 (U5) computing
/CS0 OR /CS3. The 245 now drives the bus only while the TIA is selected,
so it cannot fight the ROM or the RIOT on a CPU read - which the previous
arrangement relied on the FPGA to get right.

That lands rev A at exactly 29 pins with nothing spare. Chroma (F_COL)
and the four paddle inputs do not fit and are left open at the socket;
the README documents the three ways to recover pins, the intended rev B
fix being a local 1.8 V LDO plus a fourth buffer to reclaim J6/2-9.

fpga/tia_fpga.cst now carries real pin numbers instead of TODOs, plus the
full header map and a note that pin 56 is a general I/O rather than a
dedicated clock input - the only dedicated one, PIN52/XTAL_IN, is not
brought out to the headers.

ERC is now clean: 0 violations.

Co-Authored-By: Claude Opus 5 <noreply@anthropic.com>
Parts:
- removed J1: Tang Nano 9K row A, symbol Connector_Generic:Conn_01x20
- removed J4: Tang Nano 9K row B, symbol Connector_Generic:Conn_01x20
- removed R9: 9k1, symbol Device:R
- added C6: 100n, symbol Device:C
- added J1: Tang Nano 9K - mates J5, symbol Connector_Generic:Conn_01x24
- added J4: Tang Nano 9K - mates J6, symbol Connector_Generic:Conn_01x24
- added U5: 74LVC1G32, symbol 74xGxx:74LVC1G32
Connections:
- net F_DBUS_DIR is gone; now on net F_RW: U2.1 (A->B)
- net +3V3: now also C6.1, J4.24 (Pin_24), U5.5 (VCC)
- net F_A0: now also J1.11 (Pin_11)
- net F_A1: now also J1.12 (Pin_12)
- net F_A2: now also J1.13 (Pin_13)
- net F_A3: now also J1.14 (Pin_14)
- net F_A4: now also J1.15 (Pin_15)
- net F_A5: now also J1.16 (Pin_16)
- net F_AU0: now also J4.22 (Pin_22)
- net F_AU1: now also J1.3 (Pin_3)
- net F_CS0_N: now also J1.18 (Pin_18), U5.1
- net F_CS3_N: now also J1.19 (Pin_19), U5.2
- net F_CSYNC: now also J4.11 (Pin_11)
- net F_D0: now also U2.2 (A0), J1.5 (Pin_5); no longer U2.18 (B0)
- net F_D1: now also U2.3 (A1), J1.6 (Pin_6); no longer U2.17 (B1)
- net F_D2: now also U2.4 (A2), J1.7 (Pin_7); no longer U2.16 (B2)
- net F_D3: now also U2.5 (A3), J1.8 (Pin_8); no longer U2.15 (B3)
- net F_D4: now also U2.6 (A4), J1.9 (Pin_9); no longer U2.14 (B4)
- net F_D5: now also U2.7 (A5), J1.10 (Pin_10); no longer U2.13 (B5)
- net F_D6: now also U2.8 (A6), J1.1 (Pin_1); no longer U2.12 (B6)
- net F_D7: now also U2.9 (A7), J1.2 (Pin_2); no longer U2.11 (B7)
- net F_I4: now also J1.4 (Pin_4)
- net F_I5: now also J4.10 (Pin_10)
- net F_LUM0: now also J4.19 (Pin_19)
- net F_LUM1: now also J4.20 (Pin_20)
- net F_LUM2: now also J4.21 (Pin_21)
- net F_OSC: now also J1.21 (Pin_21)
- net F_PHI0: now also J1.22 (Pin_22)
- net F_PHI2: now also J1.20 (Pin_20)
- net F_RDY: now also J4.1 (Pin_1)
- net F_RW: now also J1.17 (Pin_17)
- net GND: now also C6.2, J4.23 (Pin_23), U5.3 (GND)
- net TIA_D0: now also U2.18 (B0); no longer U2.2 (A0)
- net TIA_D1: now also U2.17 (B1); no longer U2.3 (A1)
- net TIA_D2: now also U2.16 (B2); no longer U2.4 (A2)
- net TIA_D3: now also U2.15 (B3); no longer U2.5 (A3)
- net TIA_D4: now also U2.14 (B4); no longer U2.6 (A4)
- net TIA_D5: now also U2.13 (B5); no longer U2.7 (A5)
- net TIA_D6: now also U2.12 (B6); no longer U2.8 (A6)
- net TIA_D7: now also U2.11 (B7); no longer U2.9 (A7)
- net F_COL: no longer names the net of J2.9 (Pin_9)
- net F_DBUS_OE_N renamed DBUS_OE_N
- net DBUS_OE_N: now also U5.4
- net TIA_I0: no longer names the net of J3.20 (Pin_20)
- net TIA_I1: no longer names the net of J3.19 (Pin_19)
- net TIA_I2: no longer names the net of J3.18 (Pin_18)
- net TIA_I3: no longer names the net of J3.17 (Pin_17)
- no-connect marks 7 -> 29
Other:
- note added: "+3V3 comes from the Tang Nano (J4/24). +5 V comes from the breadboard rail."
- note added: "1.8 V-powered buffer. Recovering those 8 pins is the rev B fix."
- note added: "8 are HDMI differential pairs, 3 are power. Rev A uses all 29, with none spare."
- note added: "J4/18 (+5 V from the Tang Nano) left open on purpose: this board is fed"
- note added: "J4/2-9 are BANK3 at 1.8 V - unusable at 3.3 V without a local LDO and a"
- note added: "Of the 48 header pins only 29 are usable 3.3 V GPIO: 8 are BANK3 at 1.8 V,"
- note added: "Pin 9 (COL, chroma) and pins 37-40 (paddles) left open:"
- note added: "Pin map verified against both Sipeed board revisions (3672 and 3674), which agree."
- note added: "Power the Tang Nano over USB. +3V3 is taken from J4/24."
- note added: "Rev A - digital interface only. Chroma and paddles do not fit the pin budget; see the notes."
- note added: "U2 D0-D7. A side = FPGA, B side = TIA, so DIR can be driven straight from"
- note added: "U5 /OE = /CS0 OR /CS3. The 245 drives the bus only while the TIA is"
- note added: "budget was short by."
- note added: "from the breadboard rail, so tying both would put two sources on one net."
- note added: "keeps both 245 control lines off the FPGA - saving the one pin the header"
- note added: "no FPGA pin is left for them on a Tang Nano 9K. See README."
- note added: "selected, so it never fights the ROM or the RIOT on a CPU read."
- note added: "the buffered R/W: DIR=1 (read) sends FPGA -> TIA. That, plus the U5 gate,"
- note removed: "+3V3 comes from the Tang Nano itself. +5 V comes from the breadboard rail."
- note removed: "FPGA pin assignment lives in fpga/tia_fpga.cst - see the TODOs there."
- note removed: "Header numbering follows the Sipeed silkscreen."
- note removed: "Rev A - digital interface only. Composite video and paddles are deferred to later revisions."
- note removed: "U2 D0-D7 bidirectional. DIR=1 -> A(TIA) to B(FPGA) = CPU write."
- note removed: "Vcc is 3.3 V: LVC inputs tolerate the 6507's 5 V swing."

Commit message: Add HDMI colour output, fix schematic text collisions, correct author name
Colour video:

The chroma pin (TIA pin 9) has no FPGA pin left on a Tang Nano 9K, so the
composite output is monochrome — 8 grey levels, correct sync, everything
else intact. Colour instead comes out of the Tang Nano's own HDMI
connector: the 7-bit colour value never leaves the FPGA, and the HDMI
pins are dedicated differential pairs that were never part of the 29-pin
GPIO budget, so colour costs zero header pins.

Documented in the schematic with the TMDS pin numbers (CK 69/68, D0
71/70, D1 73/72, D2 75/74) and a design rule: J1/23-24 and J4/12-17 must
stay open, because those header pins carry the same differential pairs
and any stub attached to them degrades the signal. They were already
marked no-connect; now it is on purpose rather than by omission.

Schematic legibility:

Reference and value text was placed at fixed offsets from each symbol's
pin extents, which put it on top of bodies and net labels — worst on the
74AHCT125, whose triangle rises above its own pin row, and on every part
with a VCC pin whose label runs upward.

Placement is now searched rather than assumed. The generator tracks
occupied rectangles for symbol bodies, net labels and note text, and
drops each reference/value into the first candidate position that is
actually free. Symbol outlines come from the drawn graphics, not just
the pins.

Also moved the power symbols away from U3, where the GND symbol sat
beside the G1/G2 pins and read as an orphan, and gave the middle column
and the video resistor network enough room that labels no longer collide.

ERC: 0 violations.

Author name corrected to Leonardo Roman da Rosa in the schematic title
block, the copyright note, the README and the constraint file. The
GitHub URL keeps the lrrosa account handle.

Also ignore KiCad 10's .history/ local-history store, which is a nested
git repository and broke staging.

Co-Authored-By: Claude Opus 5 <noreply@anthropic.com>
Other:
- note added: "COLOUR VIDEO - via the Tang Nano's HDMI connector"
- note added: "Copyright 2026 Leonardo Roman da Rosa - SPDX-License-Identifier: CERN-OHL-S-2.0"
- note added: "DIR comes straight from the buffered R/W: DIR=1 (a read)"
- note added: "FPGA pins (P/N): CK 69/68, D0 71/70, D1 73/72, D2 75/74."
- note added: "RULE: leave J1/23-24 and J4/12-17 open - they carry the"
- note added: "TMDS encoder drives the HDMI pins, which are dedicated"
- note added: "The 7-bit colour value never leaves the FPGA: an internal"
- note added: "U2 D0-D7 bidirectional. A side = FPGA, B side = TIA."
- note added: "control line costs an FPGA pin - that freed the one we needed."
- note added: "differential pairs on the module and were never part of"
- note added: "same TMDS pairs, and any stub degrades the signal."
- note added: "sends FPGA -> TIA. /OE comes from U5, so neither 245"
- note added: "the 29-pin GPIO budget. Colour costs zero header pins."
- note removed: "Copyright 2026 lrrosa - SPDX-License-Identifier: CERN-OHL-S-2.0"
- note removed: "U2 D0-D7. A side = FPGA, B side = TIA, so DIR can be driven straight from"
- note removed: "budget was short by."
- note removed: "keeps both 245 control lines off the FPGA - saving the one pin the header"
- note removed: "the buffered R/W: DIR=1 (read) sends FPGA -> TIA. That, plus the U5 gate,"
- company: lrrosa - CERN-OHL-S-2.0 -> Leonardo Roman da Rosa - CERN-OHL-S-2.0

Commit message: Add rev A PCB: footprints, placement, autorouting, fabrication output
The schematic had no footprints and there was no board at all, so this adds
the whole chain rather than just a routing pass.

Footprints are SOIC/0805 throughout. That is forced rather than chosen: the
74LVC245A and 74LVC541A have no DIP version, so through-hole would have meant
soldering adapter boards onto the PCB.

Board is a 72 x 100 mm two-layer sandwich — Tang Nano sockets at the top, the
TIA's DIP-40 pins at the bottom, logic in between. Placement centres each
connector on its pad bounding box rather than trusting footprint rotation
conventions, which is also what gets J3 right: it needs pin 1 at the opposite
end from J2, because DIP pin 21 sits across from pin 20.

Routed with Freerouting 2.2.4 through the decoy-board flow: outline pulled
0.35 mm inward so copper ends up clear of the real edge, netclasses read from
the project file (0.25 mm signal, 0.6 mm power, 0.15 mm clearance). All 109
connections routed in 19 s over 6 passes; 736 segments, 61 vias, 3.72 m of
copper.

kicad-cli DRC: 0 violations, 0 unconnected items.

Gerber X2 and Excellon drill output in gerbers/.

Two things the README now flags, because they matter before anyone orders a
board:

- The Tang Nano 9K header row spacing is DEDUCED, not measured. Sipeed gives
  the module as 70 x 26 mm at 2.54 mm pitch but does not publish the row
  spacing; 20.32 mm is the only value that leaves sensible pad-to-edge
  clearance on a 26 mm board. Check it with a caliper. The DIP-40 spacing is
  fixed by the package and is not a guess.
- There is no ground pour, and placement does not follow connector pin order,
  so the buses cross the board diagonally. Both are rev B work.

Co-Authored-By: Claude Opus 5 <noreply@anthropic.com>
Parts:
- C1, C2, C3, C4, C5, C6: footprint (none) -> Capacitor_SMD:C_0805_2012Metric
- J1, J4: footprint (none) -> Connector_PinSocket_2.54mm:PinSocket_1x24_P2.54mm_Vertical
- J2, J3: footprint (none) -> Connector_PinHeader_2.54mm:PinHeader_1x20_P2.54mm_Vertical
- R1, R2, R3, R4, R5, R6, R7, R8: footprint (none) -> Resistor_SMD:R_0805_2012Metric
- U1: footprint (none) -> Package_SO:SOIC-14_3.9x8.7mm_P1.27mm
- U2, U3, U4: footprint (none) -> Package_SO:SOIC-20W_7.5x12.8mm_P1.27mm
- U5: footprint (none) -> Package_TO_SOT_SMD:SOT-23-5
Changed lines of the file:
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@@
 			)
 		)
-		(property "Footprint" ""
+		(property "Footprint" "Connector_PinSocket_2.54mm:PinSocket_1x24_P2.54mm_Vertical"
 			(at 44.45 100.33 0)
 			(hide yes)
@@
 		(instances
 			(project "tia-fpga"
-				(path "/3b635726-b7b9-42f2-b0e7-41170b4e11b6"
+				(path "/5f598ce8-ca6a-4129-874a-bfed97976bf2"
 					(reference "J1")
 					(unit 1)
@@
 			)
 		)
-		(property "Footprint" ""
+		(property "Footprint" "Connector_PinSocket_2.54mm:PinSocket_1x24_P2.54mm_Vertical"
 			(at 90.17 100.33 0)
 			(hide yes)
@@
 		(instances
 			(project "tia-fpga"
-				(path "/3b635726-b7b9-42f2-b0e7-41170b4e11b6"
+				(path "/5f598ce8-ca6a-4129-874a-bfed97976bf2"
 					(reference "J4")
 					(unit 1)
@@
 			)
 		)
-		(property "Footprint" ""
+		(property "Footprint" "Package_SO:SOIC-14_3.9x8.7mm_P1.27mm"
 			(at 165.10 55.88 0)
 			(hide yes)
@@
 		(instances
 			(project "tia-fpga"
-				(path "/3b635726-b7b9-42f2-b0e7-41170b4e11b6"
+				(path "/5f598ce8-ca6a-4129-874a-bfed97976bf2"
 					(reference "U1")
 					(unit 1)
@@
 			)
 		)
-		(property "Footprint" ""
+		(property "Footprint" "Package_SO:SOIC-14_3.9x8.7mm_P1.27mm"
 			(at 165.10 77.47 0)
 			(hide yes)
@@
 		(instances
 			(project "tia-fpga"
-				(path "/3b635726-b7b9-42f2-b0e7-41170b4e11b6"
+				(path "/5f598ce8-ca6a-4129-874a-bfed97976bf2"
 					(reference "U1")
 					(unit 2)
@@
 			)
 		)
-		(property "Footprint" ""
+		(property "Footprint" "Package_SO:SOIC-14_3.9x8.7mm_P1.27mm"
 			(at 165.10 100.33 0)
 			(hide yes)
@@
 		(instances
 			(project "tia-fpga"
-				(path "/3b635726-b7b9-42f2-b0e7-41170b4e11b6"
+				(path "/5f598ce8-ca6a-4129-874a-bfed97976bf2"
 					(reference "U1")
 					(unit 3)
@@
 			)
 		)
-		(property "Footprint" ""
+		(property "Footprint" "Package_SO:SOIC-14_3.9x8.7mm_P1.27mm"
 			(at 165.10 121.92 0)
 			(hide yes)
@@
 		(instances
 			(project "tia-fpga"
-				(path "/3b635726-b7b9-42f2-b0e7-41170b4e11b6"
+				(path "/5f598ce8-ca6a-4129-874a-bfed97976bf2"
 					(reference "U1")
 					(unit 4)
@@
 			)
 		)
-		(property "Footprint" ""
+		(property "Footprint" "Package_SO:SOIC-14_3.9x8.7mm_P1.27mm"
 			(at 209.55 55.88 0)
 			(hide yes)
@@
 		(instances
 			(project "tia-fpga"
-				(path "/3b635726-b7b9-42f2-b0e7-41170b4e11b6"
+				(path "/5f598ce8-ca6a-4129-874a-bfed97976bf2"
 					(reference "U1")
 					(unit 5)
@@
 			)
 		)
-		(property "Footprint" ""
+		(property "Footprint" "Package_SO:SOIC-20W_7.5x12.8mm_P1.27mm"
 			(at 165.10 185.42 0)
 			(hide yes)
@@
 		(instances
 			(project "tia-fpga"
-				(path "/3b635726-b7b9-42f2-b0e7-41170b4e11b6"
+				(path "/5f598ce8-ca6a-4129-874a-bfed97976bf2"
 					(reference "U2")
 					(unit 1)
@@
 			)
 		)
-		(property "Footprint" ""
+		(property "Footprint" "Package_TO_SOT_SMD:SOT-23-5"
 			(at 250.19 170.18 0)
 			(hide yes)
@@
 		(instances
 			(project "tia-fpga"
-				(path "/3b635726-b7b9-42f2-b0e7-41170b4e11b6"
+				(path "/5f598ce8-ca6a-4129-874a-bfed97976bf2"
 					(reference "U5")
 					(unit 1)
@@
 			)
 		)
-		(property "Footprint" ""
+		(property "Footprint" "Package_SO:SOIC-20W_7.5x12.8mm_P1.27mm"
 			(at 165.10 246.38 0)
 			(hide yes)
@@
 		(instances
 			(project "tia-fpga"
-				(path "/3b635726-b7b9-42f2-b0e7-41170b4e11b6"
+				(path "/5f598ce8-ca6a-4129-874a-bfed97976bf2"
 					(reference "U3")
 					(unit 1)
@@
 			)
 		)
-		(property "Footprint" ""
+		(property "Footprint" "Package_SO:SOIC-20W_7.5x12.8mm_P1.27mm"
 			(at 275.59 246.38 0)
 			(hide yes)
@@
 		(instances
 			(project "tia-fpga"
-				(path "/3b635726-b7b9-42f2-b0e7-41170b4e11b6"
+				(path "/5f598ce8-ca6a-4129-874a-bfed97976bf2"
 					(reference "U4")
 					(unit 1)
@@
 			)
 		)
-		(property "Footprint" ""
+		(property "Footprint" "Connector_PinHeader_2.54mm:PinHeader_1x20_P2.54mm_Vertical"
 			(at 355.60 95.25 0)
 			(hide yes)
@@
 		(instances
 			(project "tia-fpga"
-				(path "/3b635726-b7b9-42f2-b0e7-41170b4e11b6"
+				(path "/5f598ce8-ca6a-4129-874a-bfed97976bf2"
 					(reference "J2")
 					(unit 1)
@@
 			)
 		)
-		(property "Footprint" ""
+		(property "Footprint" "Connector_PinHeader_2.54mm:PinHeader_1x20_P2.54mm_Vertical"
 			(at 394.97 95.25 0)
 			(hide yes)
@@
 		(instances
 			(project "tia-fpga"
-				(path "/3b635726-b7b9-42f2-b0e7-41170b4e11b6"
+				(path "/5f598ce8-ca6a-4129-874a-bfed97976bf2"
 					(reference "J3")
 					(unit 1)
@@
 			)
 		)
-		(property "Footprint" ""
+		(property "Footprint" "Resistor_SMD:R_0805_2012Metric"
 			(at 330.20 187.96 0)
 			(hide yes)
@@
 		(instances
 			(project "tia-fpga"
-				(path "/3b635726-b7b9-42f2-b0e7-41170b4e11b6"
+				(path "/5f598ce8-ca6a-4129-874a-bfed97976bf2"
 					(reference "R1")
 					(unit 1)
@@
 			)
 		)
-		(property "Footprint" ""
+		(property "Footprint" "Resistor_SMD:R_0805_2012Metric"
 			(at 351.79 187.96 0)
 			(hide yes)
@@
 		(instances
 			(project "tia-fpga"
-				(path "/3b635726-b7b9-42f2-b0e7-41170b4e11b6"
+				(path "/5f598ce8-ca6a-4129-874a-bfed97976bf2"
 					(reference "R2")
 					(unit 1)
@@
 			)
 		)
-		(property "Footprint" ""
+		(property "Footprint" "Resistor_SMD:R_0805_2012Metric"
 			(at 373.38 187.96 0)
 			(hide yes)
@@
 		(instances
 			(project "tia-fpga"
-				(path "/3b635726-b7b9-42f2-b0e7-41170b4e11b6"
+				(path "/5f598ce8-ca6a-4129-874a-bfed97976bf2"
 					(reference "R3")
 					(unit 1)
@@
 			)
 		)
-		(property "Footprint" ""
+		(property "Footprint" "Resistor_SMD:R_0805_2012Metric"
 			(at 396.24 187.96 0)
 			(hide yes)
@@
 		(instances
 			(project "tia-fpga"
-				(path "/3b635726-b7b9-42f2-b0e7-41170b4e11b6"
+				(path "/5f598ce8-ca6a-4129-874a-bfed97976bf2"
 					(reference "R4")
 					(unit 1)
@@
 			)
 		)
-		(property "Footprint" ""
+		(property "Footprint" "Resistor_SMD:R_0805_2012Metric"
 			(at 330.20 213.36 0)
 			(hide yes)
@@
 		(instances
 			(project "tia-fpga"
-				(path "/3b635726-b7b9-42f2-b0e7-41170b4e11b6"
+				(path "/5f598ce8-ca6a-4129-874a-bfed97976bf2"
 					(reference "R5")
 					(unit 1)
@@
 			)
 		)
-		(property "Footprint" ""
+		(property "Footprint" "Resistor_SMD:R_0805_2012Metric"
 			(at 351.79 213.36 0)
 			(hide yes)
@@
 		(instances
 			(project "tia-fpga"
-				(path "/3b635726-b7b9-42f2-b0e7-41170b4e11b6"
+				(path "/5f598ce8-ca6a-4129-874a-bfed97976bf2"
 					(reference "R6")
 					(unit 1)
@@
 			)
 		)
-		(property "Footprint" ""
+		(property "Footprint" "Resistor_SMD:R_0805_2012Metric"
 			(at 373.38 213.36 0)
 			(hide yes)
@@
 		(instances
 			(project "tia-fpga"
-				(path "/3b635726-b7b9-42f2-b0e7-41170b4e11b6"
+				(path "/5f598ce8-ca6a-4129-874a-bfed97976bf2"
 					(reference "R7")
 					(unit 1)
@@
 			)
 		)
-		(property "Footprint" ""
+		(property "Footprint" "Resistor_SMD:R_0805_2012Metric"
 			(at 396.24 213.36 0)
 			(hide yes)
@@
 		(instances
 			(project "tia-fpga"
-				(path "/3b635726-b7b9-42f2-b0e7-41170b4e11b6"
+				(path "/5f598ce8-ca6a-4129-874a-bfed97976bf2"
 					(reference "R8")
 					(unit 1)
@@
 			)
 		)
-		(property "Footprint" ""
+		(property "Footprint" "Capacitor_SMD:C_0805_2012Metric"
 			(at 30.48 218.44 0)
 			(hide yes)
@@
 		(instances
 			(project "tia-fpga"
-				(path "/3b635726-b7b9-42f2-b0e7-41170b4e11b6"
+				(path "/5f598ce8-ca6a-4129-874a-bfed97976bf2"
 					(reference "C1")
 					(unit 1)
@@
 			)
 		)
-		(property "Footprint" ""
+		(property "Footprint" "Capacitor_SMD:C_0805_2012Metric"
 			(at 49.53 218.44 0)
 			(hide yes)
@@
 		(instances
 			(project "tia-fpga"
-				(path "/3b635726-b7b9-42f2-b0e7-41170b4e11b6"
+				(path "/5f598ce8-ca6a-4129-874a-bfed97976bf2"
 					(reference "C2")
 					(unit 1)
@@
 			)
 		)
-		(property "Footprint" ""
+		(property "Footprint" "Capacitor_SMD:C_0805_2012Metric"
 			(at 69.85 218.44 0)
 			(hide yes)
@@
 		(instances
 			(project "tia-fpga"
-				(path "/3b635726-b7b9-42f2-b0e7-41170b4e11b6"
+				(path "/5f598ce8-ca6a-4129-874a-bfed97976bf2"
 					(reference "C3")
 					(unit 1)
@@
 			)
 		)
-		(property "Footprint" ""
+		(property "Footprint" "Capacitor_SMD:C_0805_2012Metric"
 			(at 90.17 218.44 0)
 			(hide yes)
@@
 		(instances
 			(project "tia-fpga"
-				(path "/3b635726-b7b9-42f2-b0e7-41170b4e11b6"
+				(path "/5f598ce8-ca6a-4129-874a-bfed97976bf2"
 					(reference "C4")
 					(unit 1)
@@
 			)
 		)
-		(property "Footprint" ""
+		(property "Footprint" "Capacitor_SMD:C_0805_2012Metric"
 			(at 110.49 218.44 0)
 			(hide yes)
@@
 		(instances
 			(project "tia-fpga"
-				(path "/3b635726-b7b9-42f2-b0e7-41170b4e11b6"
+				(path "/5f598ce8-ca6a-4129-874a-bfed97976bf2"
 					(reference "C5")
 					(unit 1)
@@
 			)
 		)
-		(property "Footprint" ""
+		(property "Footprint" "Capacitor_SMD:C_0805_2012Metric"
 			(at 129.54 218.44 0)
 			(hide yes)
@@
 		(instances
 			(project "tia-fpga"
-				(path "/3b635726-b7b9-42f2-b0e7-41170b4e11b6"
+				(path "/5f598ce8-ca6a-4129-874a-bfed97976bf2"
 					(reference "C6")
 					(unit 1)
@@
 		(instances
 			(project "tia-fpga"
-				(path "/3b635726-b7b9-42f2-b0e7-41170b4e11b6"
+				(path "/5f598ce8-ca6a-4129-874a-bfed97976bf2"
 					(reference "#FLG1")
 					(unit 1)
@@
 		(instances
 			(project "tia-fpga"
-				(path "/3b635726-b7b9-42f2-b0e7-41170b4e11b6"
+				(path "/5f598ce8-ca6a-4129-874a-bfed97976bf2"
 					(reference "#FLG2")
 					(unit 1)
@@
 		(instances
 			(project "tia-fpga"
-				(path "/3b635726-b7b9-42f2-b0e7-41170b4e11b6"
+				(path "/5f598ce8-ca6a-4129-874a-bfed97976bf2"
 					(reference "#FLG3")
 					(unit 1)
@@
 		(instances
 			(project "tia-fpga"
-				(path "/3b635726-b7b9-42f2-b0e7-41170b4e11b6"
+				(path "/5f598ce8-ca6a-4129-874a-bfed97976bf2"
 					(reference "#PWR1")
 					(unit 1)
@@
 		(instances
 			(project "tia-fpga"
-				(path "/3b635726-b7b9-42f2-b0e7-41170b4e11b6"
+				(path "/5f598ce8-ca6a-4129-874a-bfed97976bf2"
 					(reference "#PWR2")
 					(unit 1)
@@
 		(instances
 			(project "tia-fpga"
-				(path "/3b635726-b7b9-42f2-b0e7-41170b4e11b6"
+				(path "/5f598ce8-ca6a-4129-874a-bfed97976bf2"
 					(reference "#PWR3")
 					(unit 1)
