File: tia-fpga.kicad_sch (KiCad schematic)
At the start: 23 parts, among them J1 Tang Nano 9K - mates J5, J2 TIA pins 1-20, J3 TIA pins 21-40, J4 Tang Nano 9K - mates J6, U1 74AHCT125, U2 74LVC245A, U3 74LVC541A, U4 74LVC541A, U5 74LVC1G32

Commit message: Put the TIA pins on the back, add mounting holes and a ground pour, fit chroma
Four changes, one of them a real bug.

THE BUG: all four connectors were on the front. The Tang Nano sockets and
the TIA pin headers were mounted on the same side, which means the board
could never have gone into a socket — the pins pointed up alongside the
sockets instead of down. J2/J3 now sit on B.Cu. Flipping mirrors the pad
order, so the placement loop checks which end pin 1 landed on and spins
the part 180 degrees about its own pad centre when it is wrong; J2 keeps
pin 1 at the left, J3 at the right, preserving the DIP-40 wrap-around.

This also removed the nine courtyard overlaps for free: with the headers
on the back and the SMD logic on the front, they no longer share space,
so KiCad's generous SOIC courtyard has nothing to collide with.

CHROMA IS BACK. F_COL took the pin that carried PHI2. The trade is sound:
the FPGA generates PHI0 itself, so it knows where it is in the bus cycle
and can time accesses from its own clock rather than the 6507's output.
It costs a little timing fidelity and buys back colour on the composite
and RF path. That matters because the likeliest use of this board is not
a bench rig — it is reviving a console with a dead TIA while keeping its
original video. R9 comes back with it, and the README now spells out that
R1-R9 must be left unpopulated in a real 2600, where the console already
has that ladder and a second one in parallel would shift every level.
PHI2 is still buffered by U3 and brought to an unconnected pad.

MOUNTING HOLES: four M2 in the corners. The board grew to 76 x 36 mm to
make room for them without crowding the connector rows.

GROUND POUR: 1418 mm2 on B.Cu, filled after routing. It has to be after —
Freerouting reads a pour as an obstacle and goes effectively single-layer
with one present.

Routing needed one more perturbation than before: 0.15 mm clearance left
F_I5 unrouted, 0.13 mm routed all 111 connections in 22.6 s. 758
segments, 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
Parts:
- added R9: 9k1, Resistor_SMD:R_0805_2012Metric, symbol Device:R
Connections:
- net VIDEO_SUM: now also R9.2
- net F_COL: now reaches J2.9 (Pin_9)
- net F_COL: now also J1.20 (Pin_20), R9.1
- net F_PHI2: no longer names the net of U3.11 (Y7)
- net F_PHI2: no longer J1.20 (Pin_20)
Other:
- note added: "4:2:1 luma weighting, plus R9 for chroma. Do NOT populate when the board"
- note added: "VIDEO OUTPUT - CX-2600A resistor network (STANDALONE USE ONLY)"
- note added: "goes into a real 2600: the console already has this network, and a second"
- note added: "one in parallel would shift every level. Drive the socket pins and stop."
- note removed: "4:2:1 luma weighting. Output stage (2N3563) follows the original sheet."
- note removed: "VIDEO OUTPUT - CX-2600A resistor network (phase 6, not populated)"
Changed lines of the file:
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@@
 		(instances
 			(project "tia-fpga"
-				(path "/5f598ce8-ca6a-4129-874a-bfed97976bf2"
+				(path "/2e306981-9160-43af-a437-b150d51b2219"
 					(reference "J1")
 					(unit 1)
@@
 		)
 	)
-	(label "F_PHI2"
+	(label "F_COL"
 		(at 36.83 120.65 0)
 		(effects
@@
 		(instances
 			(project "tia-fpga"
-				(path "/5f598ce8-ca6a-4129-874a-bfed97976bf2"
+				(path "/2e306981-9160-43af-a437-b150d51b2219"
 					(reference "J4")
 					(unit 1)
@@
 		(instances
 			(project "tia-fpga"
-				(path "/5f598ce8-ca6a-4129-874a-bfed97976bf2"
+				(path "/2e306981-9160-43af-a437-b150d51b2219"
 					(reference "U1")
 					(unit 1)
@@
 		(instances
 			(project "tia-fpga"
-				(path "/5f598ce8-ca6a-4129-874a-bfed97976bf2"
+				(path "/2e306981-9160-43af-a437-b150d51b2219"
 					(reference "U1")
 					(unit 2)
@@
 		(instances
 			(project "tia-fpga"
-				(path "/5f598ce8-ca6a-4129-874a-bfed97976bf2"
+				(path "/2e306981-9160-43af-a437-b150d51b2219"
 					(reference "U1")
 					(unit 3)
@@
 		(instances
 			(project "tia-fpga"
-				(path "/5f598ce8-ca6a-4129-874a-bfed97976bf2"
+				(path "/2e306981-9160-43af-a437-b150d51b2219"
 					(reference "U1")
 					(unit 4)
@@
 		(instances
 			(project "tia-fpga"
-				(path "/5f598ce8-ca6a-4129-874a-bfed97976bf2"
+				(path "/2e306981-9160-43af-a437-b150d51b2219"
 					(reference "U1")
 					(unit 5)
@@
 		(instances
 			(project "tia-fpga"
-				(path "/5f598ce8-ca6a-4129-874a-bfed97976bf2"
+				(path "/2e306981-9160-43af-a437-b150d51b2219"
 					(reference "U2")
 					(unit 1)
@@
 		(instances
 			(project "tia-fpga"
-				(path "/5f598ce8-ca6a-4129-874a-bfed97976bf2"
+				(path "/2e306981-9160-43af-a437-b150d51b2219"
 					(reference "U5")
 					(unit 1)
@@
 		(instances
 			(project "tia-fpga"
-				(path "/5f598ce8-ca6a-4129-874a-bfed97976bf2"
+				(path "/2e306981-9160-43af-a437-b150d51b2219"
 					(reference "U3")
 					(unit 1)
@@
 		)
 	)
-	(wire
-		(pts
-			(xy 177.80 251.46) (xy 180.34 251.46)
-		)
-		(stroke
-			(width 0)
-			(type default)
-		)
-	)
-	(label "F_PHI2"
-		(at 180.34 251.46 0)
-		(effects
-			(font
-				(size 1.27 1.27)
-			)
-			(justify left bottom)
-		)
+	(no_connect
+		(at 177.80 251.46)
 	)
 	(wire
@@
 		(instances
 			(project "tia-fpga"
-				(path "/5f598ce8-ca6a-4129-874a-bfed97976bf2"
+				(path "/2e306981-9160-43af-a437-b150d51b2219"
 					(reference "U4")
 					(unit 1)
@@
 		(instances
 			(project "tia-fpga"
-				(path "/5f598ce8-ca6a-4129-874a-bfed97976bf2"
+				(path "/2e306981-9160-43af-a437-b150d51b2219"
 					(reference "J2")
 					(unit 1)
@@
 		)
 	)
-	(no_connect
-		(at 350.52 92.71)
+	(wire
+		(pts
+			(xy 350.52 92.71) (xy 347.98 92.71)
+		)
+		(stroke
+			(width 0)
+			(type default)
+		)
+	)
+	(label "F_COL"
+		(at 347.98 92.71 0)
+		(effects
+			(font
+				(size 1.27 1.27)
+			)
+			(justify right bottom)
+		)
 	)
 	(no_connect
@@
 		(instances
 			(project "tia-fpga"
-				(path "/5f598ce8-ca6a-4129-874a-bfed97976bf2"
+				(path "/2e306981-9160-43af-a437-b150d51b2219"
 					(reference "J3")
 					(unit 1)
@@
 		)
 	)
-	(text "VIDEO OUTPUT - CX-2600A resistor network (phase 6, not populated)"
+	(text "VIDEO OUTPUT - CX-2600A resistor network (STANDALONE USE ONLY)"
 		(exclude_from_sim no)
-		(at 300.00 168.00 0)
+		(at 300.00 164.00 0)
 		(effects
 			(font
@@
 		)
 	)
-	(text "4:2:1 luma weighting. Output stage (2N3563) follows the original sheet."
+	(text "4:2:1 luma weighting, plus R9 for chroma. Do NOT populate when the board"
 		(exclude_from_sim no)
-		(at 300.00 172.00 0)
+		(at 300.00 168.00 0)
+		(effects
+			(font
+				(size 1.30 1.30)
+			)
+			(justify left)
+		)
+	)
+	(text "goes into a real 2600: the console already has this network, and a second"
+		(exclude_from_sim no)
+		(at 300.00 171.50 0)
+		(effects
+			(font
+				(size 1.30 1.30)
+			)
+			(justify left)
+		)
+	)
+	(text "one in parallel would shift every level. Drive the socket pins and stop."
+		(exclude_from_sim no)
+		(at 300.00 175.00 0)
 		(effects
 			(font
@@
 		(instances
 			(project "tia-fpga"
-				(path "/5f598ce8-ca6a-4129-874a-bfed97976bf2"
+				(path "/2e306981-9160-43af-a437-b150d51b2219"
 					(reference "R1")
 					(unit 1)
@@
 		(instances
 			(project "tia-fpga"
-				(path "/5f598ce8-ca6a-4129-874a-bfed97976bf2"
+				(path "/2e306981-9160-43af-a437-b150d51b2219"
 					(reference "R2")
 					(unit 1)
@@
 		(instances
 			(project "tia-fpga"
-				(path "/5f598ce8-ca6a-4129-874a-bfed97976bf2"
+				(path "/2e306981-9160-43af-a437-b150d51b2219"
 					(reference "R3")
 					(unit 1)
@@
 		(instances
 			(project "tia-fpga"
-				(path "/5f598ce8-ca6a-4129-874a-bfed97976bf2"
+				(path "/2e306981-9160-43af-a437-b150d51b2219"
 					(reference "R4")
 					(unit 1)
@@
 		(instances
 			(project "tia-fpga"
-				(path "/5f598ce8-ca6a-4129-874a-bfed97976bf2"
+				(path "/2e306981-9160-43af-a437-b150d51b2219"
 					(reference "R5")
 					(unit 1)
@@
 		(instances
 			(project "tia-fpga"
-				(path "/5f598ce8-ca6a-4129-874a-bfed97976bf2"
+				(path "/2e306981-9160-43af-a437-b150d51b2219"
 					(reference "R6")
 					(unit 1)
@@
 		(instances
 			(project "tia-fpga"
-				(path "/5f598ce8-ca6a-4129-874a-bfed97976bf2"
+				(path "/2e306981-9160-43af-a437-b150d51b2219"
 					(reference "R7")
 					(unit 1)
@@
 		(instances
 			(project "tia-fpga"
-				(path "/5f598ce8-ca6a-4129-874a-bfed97976bf2"
+				(path "/2e306981-9160-43af-a437-b150d51b2219"
 					(reference "R8")
 					(unit 1)
@@
 		)
 	)
+	(symbol
+		(lib_id "Device:R")
+		(at 417.83 187.96 0)
+		(unit 1)
+		(exclude_from_sim no)
+		(in_bom yes)
+		(on_board yes)
+		(dnp no)
+		(property "Reference" "R9"
+			(at 420.35 181.18 0)
+			(effects
+				(font
+					(size 1.27 1.27)
+				)
+				(justify left)
+			)
+		)
+		(property "Value" "9k1"
+			(at 420.35 183.28 0)
+			(effects
+				(font
+					(size 1.27 1.27)
+				)
+				(justify left)
+			)
+		)
+		(property "Footprint" "Resistor_SMD:R_0805_2012Metric"
+			(at 417.83 187.96 0)
+			(hide yes)
+			(effects
+				(font
+					(size 1.27 1.27)
+				)
+				(justify left)
+			)
+		)
+		(property "Datasheet" ""
+			(at 417.83 187.96 0)
+			(hide yes)
+			(effects
+				(font
+					(size 1.27 1.27)
+				)
+				(justify left)
+			)
+		)
+		(pin "1"
+		)
+		(pin "2"
+		)
+		(instances
+			(project "tia-fpga"
+				(path "/2e306981-9160-43af-a437-b150d51b2219"
+					(reference "R9")
+					(unit 1)
+				)
+			)
+		)
+	)
+	(wire
+		(pts
+			(xy 417.83 184.15) (xy 417.83 181.61)
+		)
+		(stroke
+			(width 0)
+			(type default)
+		)
+	)
+	(label "F_COL"
+		(at 417.83 181.61 90)
+		(effects
+			(font
+				(size 1.27 1.27)
+			)
+			(justify left bottom)
+		)
+	)
+	(wire
+		(pts
+			(xy 417.83 191.77) (xy 417.83 194.31)
+		)
+		(stroke
+			(width 0)
+			(type default)
+		)
+	)
+	(label "VIDEO_SUM"
+		(at 417.83 194.31 90)
+		(effects
+			(font
+				(size 1.27 1.27)
+			)
+			(justify right bottom)
+		)
+	)
 	(text "POWER AND DECOUPLING"
 		(exclude_from_sim no)
@@
 		(instances
 			(project "tia-fpga"
-				(path "/5f598ce8-ca6a-4129-874a-bfed97976bf2"
+				(path "/2e306981-9160-43af-a437-b150d51b2219"
 					(reference "C1")
 					(unit 1)
@@
 		(instances
 			(project "tia-fpga"
-				(path "/5f598ce8-ca6a-4129-874a-bfed97976bf2"
+				(path "/2e306981-9160-43af-a437-b150d51b2219"
 					(reference "C2")
 					(unit 1)
@@
 		(instances
 			(project "tia-fpga"
-				(path "/5f598ce8-ca6a-4129-874a-bfed97976bf2"
+				(path "/2e306981-9160-43af-a437-b150d51b2219"
 					(reference "C3")
 					(unit 1)
@@
 		(instances
 			(project "tia-fpga"
-				(path "/5f598ce8-ca6a-4129-874a-bfed97976bf2"
+				(path "/2e306981-9160-43af-a437-b150d51b2219"
 					(reference "C4")
 					(unit 1)
@@
 		(instances
 			(project "tia-fpga"
-				(path "/5f598ce8-ca6a-4129-874a-bfed97976bf2"
+				(path "/2e306981-9160-43af-a437-b150d51b2219"
 					(reference "C5")
 					(unit 1)
@@
 		(instances
 			(project "tia-fpga"
-				(path "/5f598ce8-ca6a-4129-874a-bfed97976bf2"
+				(path "/2e306981-9160-43af-a437-b150d51b2219"
 					(reference "C6")
 					(unit 1)
@@
 		(instances
 			(project "tia-fpga"
-				(path "/5f598ce8-ca6a-4129-874a-bfed97976bf2"
+				(path "/2e306981-9160-43af-a437-b150d51b2219"
 					(reference "#FLG1")
 					(unit 1)
@@
 		(instances
 			(project "tia-fpga"
-				(path "/5f598ce8-ca6a-4129-874a-bfed97976bf2"
+				(path "/2e306981-9160-43af-a437-b150d51b2219"
 					(reference "#FLG2")
 					(unit 1)
@@
 		(instances
 			(project "tia-fpga"
-				(path "/5f598ce8-ca6a-4129-874a-bfed97976bf2"
+				(path "/2e306981-9160-43af-a437-b150d51b2219"
 					(reference "#FLG3")
 					(unit 1)
@@
 		(instances
 			(project "tia-fpga"
-				(path "/5f598ce8-ca6a-4129-874a-bfed97976bf2"
+				(path "/2e306981-9160-43af-a437-b150d51b2219"
 					(reference "#PWR1")
 					(unit 1)
@@
 		(instances
 			(project "tia-fpga"
-				(path "/5f598ce8-ca6a-4129-874a-bfed97976bf2"
+				(path "/2e306981-9160-43af-a437-b150d51b2219"
 					(reference "#PWR2")
 					(unit 1)
@@
 		(instances
 			(project "tia-fpga"
-				(path "/5f598ce8-ca6a-4129-874a-bfed97976bf2"
+				(path "/2e306981-9160-43af-a437-b150d51b2219"
 					(reference "#PWR3")
 					(unit 1)
