File: tia-fpga.kicad_sch (KiCad schematic)
At the start: 23 parts, among them J1 Tang Nano 9K - mates J5, J2 TIA pins 1-20, J3 TIA pins 21-40, J4 Tang Nano 9K - mates J6, U1 74AHCT125, U2 74LVC245A, U3 74LVC541A, U4 74LVC541A, U5 74LVC1G32, U6 74LVC2G07, U7 74LVC2G07, U8 74LVC2G07, U9 74LVC2G07

Commit message: Fix the Tang Nano interface: row spacing, row order, 5 V
Sipeed's dimension drawing for the Tang Nano 9K settles two things this board
had guessed. The module's header rows are 22.86 mm apart, not 20.32, and seen
from above with the USB-C end on the left its J6 row is the upper one -- so the
sockets were the wrong way round as well. J1 now takes J6 and J4 takes J5.
Three sources agree on the order: the pin numbers on the module's underside,
the QN88's own pin order in the top-side photo of Sipeed's datasheet, and
third-party carrier boards for the module. Rev A had both errors too; nothing
was ever fabricated from either.

J1/18, the module's 5 V input, was left open on purpose for breadboard use,
with the Tang Nano powered over USB. In a console that would mean a USB supply
inside the case, so D1 (MBR0540, SOD-123) now feeds it from the TIA socket's
+5 V and blocks the module's USB from feeding the console back.

The board grows 2.54 mm, to 70 x 34.54 mm: J4 moves to y = 28.70 and the
channel's decoupling moves with it, which leaves the top margin as it was. The
pin assignment was solved again for the new geometry (571 mm summed, F_OSC
still on J6/1, the PLL's own input) and the board re-routed: 561 segments, 37
vias, 1.52 m of copper. Freerouting left two ground branches open; each is
closed with a via dropped on the track itself, where it passes over the main
island of the pour. ERC 0; DRC 0 violations, 0 unconnected pads.

Boot time: the console releases the 6507's reset 17 to 58 ms after power-up,
depending on the board revision, and PHI0 has to be running by then. At Gowin's
default 2.5 MHz the GW1NR-9 takes about 100 ms to load its bitstream from
flash, so build_gowin.tcl now asks for -loading_rate 250/8 (31.25 MHz, the
fastest the device allows in Autoboot): about 8 ms. Timing still closes, at
60.4 MHz against the 57.27 MHz clock.

Gerbers, drill, PDFs, renders, both BOMs and the README follow the board.

Co-Authored-By: Claude Opus 5 <noreply@anthropic.com>
Parts:
- added D1: MBR0540, Diode_SMD:D_SOD-123, symbol Device:D_Schottky
- renumbered J4 to J1, J1 to J4
Connections:
- net +5V: now also D1.2 (A)
- net F_A0: now also J4.11 (Pin_11); no longer J4.12 (Pin_12)
- net F_A1: now also J4.12 (Pin_12); no longer J1.11 (Pin_11)
- net F_A3: now also J4.10 (Pin_10); no longer J4.14 (Pin_14)
- net F_A4: now also J4.14 (Pin_14); no longer J4.15 (Pin_15)
- net F_A5: now also J1.21 (Pin_21); no longer J4.22 (Pin_22)
- net F_AU0: now also J1.20 (Pin_20); no longer J4.16 (Pin_16)
- net F_AU1: now also J1.19 (Pin_19); no longer J4.21 (Pin_21)
- net F_BLK: now also J4.7 (Pin_7); no longer J4.8 (Pin_8)
- net F_COL: now also J1.10 (Pin_10); no longer J4.11 (Pin_11)
- net F_CSYNC: now also J4.4 (Pin_4); no longer J4.5 (Pin_5)
- net F_D0: now also J4.17 (Pin_17); no longer J1.10 (Pin_10)
- net F_D1: now also J4.16 (Pin_16); no longer J4.18 (Pin_18)
- net F_D2: now also J4.18 (Pin_18); no longer J4.19 (Pin_19)
- net F_D3: now also J4.19 (Pin_19); no longer J1.19 (Pin_19)
- net F_D4: now also J1.22 (Pin_22); no longer J1.20 (Pin_20)
- net F_D6: now also J4.22 (Pin_22); no longer J1.21 (Pin_21)
- net F_D7: now also J4.21 (Pin_21); no longer J1.22 (Pin_22)
- net F_I4: now also J4.8 (Pin_8); no longer J4.6 (Pin_6)
- net F_LUM0: now also J1.11 (Pin_11); no longer J4.10 (Pin_10)
- net F_LUM1: now also J4.5 (Pin_5); no longer J4.4 (Pin_4)
- net F_LUM2: now also J4.6 (Pin_6); no longer J4.7 (Pin_7)
- net F_RW: now also J4.15 (Pin_15); no longer J4.17 (Pin_17)
- net TN_5V: now reaches J1.18 (Pin_18)
- net TN_5V: now also D1.1 (K)
- no-connect marks 28 -> 27
Other:
- note added: "+3V3 comes back from the module on J1/24 and powers U2-U9."
- note added: "+3V3 comes from the Tang Nano (J1/24). +5 V comes from the TIA socket, pin 20."
- note added: "J1/18 is the module's 5 V input, fed from the TIA socket through D1, so"
- note added: "J1/2-9 are BANK3 at 1.8 V - unusable at 3.3 V without a local LDO and a"
- note added: "RULE: leave J4/23-24 and J1/12-17 open - they carry the"
- note added: "the console powers the Tang Nano and its USB cannot feed the console back."
- note removed: "+3V3 comes from the Tang Nano (J4/24). +5 V comes from the breadboard rail."
- note removed: "J4/18 (+5 V from the Tang Nano) left open on purpose: this board is fed"
- note removed: "J4/2-9 are BANK3 at 1.8 V - unusable at 3.3 V without a local LDO and a"
- note removed: "Power the Tang Nano over USB. +3V3 is taken from J4/24."
- note removed: "RULE: leave J1/23-24 and J4/12-17 open - they carry the"
- note removed: "from the breadboard rail, so tying both would put two sources on one net."
Changed lines of the file:
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@@
 	(title_block
 		(title "TIA-FPGA - digital interface")
-		(date "2026-09-14")
+		(date "2026-09-15")
 		(rev "B")
 		(company "Leonardo Roman da Rosa - CERN-OHL-S-2.0")
@@
 		(on_board yes)
 		(dnp no)
-		(property "Reference" "J1"
+		(property "Reference" "J4"
 			(at 43.18 66.88 0)
 			(effects
@@
 			(project "tia-fpga"
 				(path "/b310daf3-ae03-4c4a-85d5-0b0546462b61"
-					(reference "J1")
+					(reference "J4")
 					(unit 1)
 				)
@@
 		)
 	)
-	(label "F_LUM1"
+	(label "F_CSYNC"
 		(at 36.83 80.01 0)
 		(effects
@@
 		)
 	)
-	(label "F_CSYNC"
+	(label "F_LUM1"
 		(at 36.83 82.55 0)
 		(effects
@@
 		)
 	)
-	(label "F_I4"
+	(label "F_LUM2"
 		(at 36.83 85.09 0)
 		(effects
@@
 		)
 	)
-	(label "F_LUM2"
+	(label "F_BLK"
 		(at 36.83 87.63 0)
 		(effects
@@
 		)
 	)
-	(label "F_BLK"
+	(label "F_I4"
 		(at 36.83 90.17 0)
 		(effects
@@
 		)
 	)
-	(label "F_LUM0"
+	(label "F_A3"
 		(at 36.83 95.25 0)
 		(effects
@@
 		)
 	)
-	(label "F_COL"
+	(label "F_A0"
 		(at 36.83 97.79 0)
 		(effects
@@
 		)
 	)
-	(label "F_A0"
+	(label "F_A1"
 		(at 36.83 100.33 0)
 		(effects
@@
 		)
 	)
-	(label "F_A3"
+	(label "F_A4"
 		(at 36.83 105.41 0)
 		(effects
@@
 		)
 	)
-	(label "F_A4"
+	(label "F_RW"
 		(at 36.83 107.95 0)
 		(effects
@@
 		)
 	)
-	(label "F_AU0"
+	(label "F_D1"
 		(at 36.83 110.49 0)
 		(effects
@@
 		)
 	)
-	(label "F_RW"
+	(label "F_D0"
 		(at 36.83 113.03 0)
 		(effects
@@
 		)
 	)
-	(label "F_D1"
+	(label "F_D2"
 		(at 36.83 115.57 0)
 		(effects
@@
 		)
 	)
-	(label "F_D2"
+	(label "F_D3"
 		(at 36.83 118.11 0)
 		(effects
@@
 		)
 	)
-	(label "F_AU1"
+	(label "F_D7"
 		(at 36.83 123.19 0)
 		(effects
@@
 		)
 	)
-	(label "F_A5"
+	(label "F_D6"
 		(at 36.83 125.73 0)
 		(effects
@@
 		(on_board yes)
 		(dnp no)
-		(property "Reference" "J4"
+		(property "Reference" "J1"
 			(at 88.90 66.88 0)
 			(effects
@@
 			(project "tia-fpga"
 				(path "/b310daf3-ae03-4c4a-85d5-0b0546462b61"
-					(reference "J4")
+					(reference "J1")
 					(unit 1)
 				)
@@
 		)
 	)
-	(label "F_D0"
+	(label "F_COL"
 		(at 82.55 95.25 0)
 		(effects
@@
 		)
 	)
-	(label "F_A1"
+	(label "F_LUM0"
 		(at 82.55 97.79 0)
 		(effects
@@
 		(at 85.09 113.03)
 	)
-	(no_connect
-		(at 85.09 115.57)
-	)
 	(wire
 		(pts
@@
 		)
 	)
-	(label "F_D3"
+	(label "F_AU1"
 		(at 82.55 118.11 0)
 		(effects
@@
 		)
 	)
-	(label "F_D4"
+	(label "F_AU0"
 		(at 82.55 120.65 0)
 		(effects
@@
 		)
 	)
-	(label "F_D6"
+	(label "F_A5"
 		(at 82.55 123.19 0)
 		(effects
@@
 		)
 	)
-	(label "F_D7"
+	(label "F_D4"
 		(at 82.55 125.73 0)
 		(effects
@@
 		)
 	)
-	(text "J4/2-9 are BANK3 at 1.8 V - unusable at 3.3 V without a local LDO and a"
+	(text "J1/2-9 are BANK3 at 1.8 V - unusable at 3.3 V without a local LDO and a"
 		(exclude_from_sim no)
 		(at 20.00 142.00 0)
@@
 		)
 	)
-	(text "J4/18 (+5 V from the Tang Nano) left open on purpose: this board is fed"
+	(text "J1/18 is the module's 5 V input, fed from the TIA socket through D1, so"
 		(exclude_from_sim no)
 		(at 20.00 150.00 0)
@@
 		)
 	)
-	(text "from the breadboard rail, so tying both would put two sources on one net."
+	(text "the console powers the Tang Nano and its USB cannot feed the console back."
 		(exclude_from_sim no)
 		(at 20.00 153.50 0)
@@
 		)
 	)
-	(text "Power the Tang Nano over USB. +3V3 is taken from J4/24."
+	(text "+3V3 comes back from the module on J1/24 and powers U2-U9."
 		(exclude_from_sim no)
 		(at 20.00 157.00 0)
@@
 		)
 	)
-	(text "+3V3 comes from the Tang Nano (J4/24). +5 V comes from the breadboard rail."
+	(text "+3V3 comes from the Tang Nano (J1/24). +5 V comes from the TIA socket, pin 20."
 		(exclude_from_sim no)
 		(at 20.00 200.00 0)
@@
 		)
 	)
-	(text "RULE: leave J1/23-24 and J4/12-17 open - they carry the"
+	(text "RULE: leave J4/23-24 and J1/12-17 open - they carry the"
 		(exclude_from_sim no)
 		(at 228.00 127.60 0)
@@
 		)
 	)
+	(wire
+		(pts
+			(xy 85.09 115.57) (xy 82.55 115.57)
+		)
+		(stroke
+			(width 0)
+			(type default)
+		)
+	)
+	(label "TN_5V"
+		(at 82.55 115.57 0)
+		(effects
+			(font
+				(size 1.27 1.27)
+			)
+			(justify right bottom)
+		)
+	)
+	(symbol
+		(lib_id "Device:D_Schottky")
+		(at 110.49 115.57 0)
+		(unit 1)
+		(exclude_from_sim no)
+		(in_bom yes)
+		(on_board yes)
+		(dnp no)
+		(property "Reference" "D1"
+			(at 109.22 110.49 0)
+			(effects
+				(font
+					(size 1.27 1.27)
+				)
+				(justify left)
+			)
+		)
+		(property "Value" "MBR0540"
+			(at 109.22 113.03 0)
+			(effects
+				(font
+					(size 1.27 1.27)
+				)
+				(justify left)
+			)
+		)
+		(property "Footprint" "Diode_SMD:D_SOD-123"
+			(at 110.49 115.57 0)
+			(hide yes)
+			(effects
+				(font
+					(size 1.27 1.27)
+				)
+				(justify left)
+			)
+		)
+		(property "Datasheet" ""
+			(at 110.49 115.57 0)
+			(hide yes)
+			(effects
+				(font
+					(size 1.27 1.27)
+				)
+				(justify left)
+			)
+		)
+		(pin "1"
+		)
+		(pin "2"
+		)
+		(instances
+			(project "tia-fpga"
+				(path "/b310daf3-ae03-4c4a-85d5-0b0546462b61"
+					(reference "D1")
+					(unit 1)
+				)
+			)
+		)
+	)
+	(wire
+		(pts
+			(xy 106.68 115.57) (xy 104.14 115.57)
+		)
+		(stroke
+			(width 0)
+			(type default)
+		)
+	)
+	(label "TN_5V"
+		(at 104.14 115.57 0)
+		(effects
+			(font
+				(size 1.27 1.27)
+			)
+			(justify right bottom)
+		)
+	)
+	(wire
+		(pts
+			(xy 114.30 115.57) (xy 116.84 115.57)
+		)
+		(stroke
+			(width 0)
+			(type default)
+		)
+	)
+	(label "+5V"
+		(at 116.84 115.57 0)
+		(effects
+			(font
+				(size 1.27 1.27)
+			)
+			(justify left bottom)
+		)
+	)
